File: PCB/CH32V003_CO2_Sensor.kicad_pcb (KiCad board)
At the start: 2 copper layers, 29.2 x 40.6 mm, 30 parts, among them Q1 AO3400A, SW2 SW_Push, SW3 SW_Push

Commit message: Minor adjustments plus BOM file added
Parts:
- VIB1: value Vibration Motor -> Mini Vibration Motor
- renumbered CH32V003 to CH32V3, LDO to LDO1, LiPo to LiPo1, Power to SW1
Connections:
- SW1 pad 3: VBUS -> unconnected-(SW1-C-Pad3)
Routing:
- net VBUS: track 38.6 -> 20.1 mm, vias 2 -> 0
Changed lines of the file:
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@@
   (net 50 "Net-(D3-A)")
   (net 51 "Net-(D4-K)")
+  (net 52 "unconnected-(SW1-C-Pad3)")
   (footprint "Resistor_SMD:R_0603_1608Metric" (layer "F.Cu")
     (at 148.4 68.4 180)
@@
         (effects (font (size 1 1) (thickness 0.15)))
     )
-    (fp_text value "Vibration Motor" (at 2 0.875 180) (layer "B.SilkS")
+    (fp_text value "Mini Vibration Motor" (at 2 0.875 180) (layer "B.SilkS")
         (effects (font (size 1 1) (thickness 0.15)) (justify mirror))
     )
@@
     (property "ki_keywords" "switch single-pole double-throw spdt ON-ON")
     (attr smd)
-    (fp_text reference "Power" (at 0 -3.2 90) (layer "F.SilkS")
+    (fp_text reference "SW1" (at 0 -3.2 90) (layer "F.SilkS")
         (effects (font (size 0.7 0.7) (thickness 0.12) bold))
     )
@@
       (net 28 "Net-(LDO1-EN)") (pinfunction "B") (pintype "passive"))
     (pad "3" smd rect (at 2.25 -1.43 270) (size 0.7 1.5) (layers "F.Cu" "F.Paste" "F.Mask")
-      (net 3 "VBUS") (pinfunction "C") (pintype "passive"))
+      (net 52 "unconnected-(SW1-C-Pad3)") (pinfunction "C") (pintype "passive+no_connect"))
     (model "${KICAD6_3DMODEL_DIR}/Button_Switch_SMD.3dshapes/SW_SPDT_PCM12.wrl"
       (offset (xyz 0 0 0))
@@
     (property "ki_keywords" "RISCV")
     (attr smd)
-    (fp_text reference "CH32V003" (at 4.45 -0.25 270 unlocked) (layer "F.SilkS")
+    (fp_text reference "CH32V3" (at 4.45 -0.25 270 unlocked) (layer "F.SilkS")
         (effects (font (size 0.7 0.7) (thickness 0.12)))
     )
@@
     (property "ki_keywords" "linear regulator ldo fixed positive")
     (attr smd)
-    (fp_text reference "LDO" (at 0.7 -0.05) (layer "F.SilkS")
+    (fp_text reference "LDO1" (at 0.7 -0.05) (layer "F.SilkS")
         (effects (font (size 0.7 0.7) (thickness 0.12) bold))
     )
@@
     (property "ki_keywords" "connector")
     (attr smd)
-    (fp_text reference "LiPo" (at -0.16 -7.65) (layer "B.SilkS")
+    (fp_text reference "LiPo1" (at -0.16 -7.65) (layer "B.SilkS")
         (effects (font (size 1 1) (thickness 0.15)) (justify mirror))
     )
@@
   (segment (start 150.888528 68.4) (end 156.21 63.078528) (width 0.3) (layer "F.Cu") (net 3))
   (segment (start 154.405 60.425) (end 151.96 60.425) (width 0.5) (layer "F.Cu") (net 3))
-  (segment (start 149.4 68.4) (end 150.6 67.2) (width 0.3) (layer "F.Cu") (net 3))
-  (segment (start 150.51 80.83) (end 152.67 80.83) (width 0.3) (layer "F.Cu") (net 3))
   (segment (start 156.21 62.23) (end 156.21 63) (width 0.5) (layer "F.Cu") (net 3))
-  (segment (start 152.67 80.83) (end 152.9 80.6) (width 0.3) (layer "F.Cu") (net 3))
   (segment (start 149.225 68.4) (end 149.4 68.4) (width 0.3) (layer "F.Cu") (net 3))
-  (via (at 152.9 80.6) (size 0.8) (drill 0.4) (layers "F.Cu" "B.Cu") (net 3))
-  (via (at 150.6 67.2) (size 0.8) (drill 0.4) (layers "F.Cu" "B.Cu") (net 3))
-  (segment (start 152.9 69.5) (end 150.6 67.2) (width 0.3) (layer "B.Cu") (net 3))
-  (segment (start 152.9 80.6) (end 152.9 69.5) (width 0.3) (layer "B.Cu") (net 3))
   (segment (start 154.64 72.2) (end 155.3 72.2) (width 0.5) (layer "F.Cu") (net 4))
   (segment (start 158.2 69.75) (end 158.2 68.2) (width 0.5) (layer "F.Cu") (net 4))
