File: PCB/CH32V003_CO2_Sensor.kicad_sch (KiCad schematic)
At the start: 29 parts, among them Q1 AO3400A, SW1 SW_SPDT, SW2 SW_Push, SW3 SW_Push

Commit message: Minor adjustments plus BOM file added
Parts:
- VIB1: footprint Connector_PinHeader_2.54mm:PinHeader_1x02_P2.54mm_Vertical -> Connector_PinSocket_2.54mm:PinSocket_1x02_P2.54mm_Vertical
Connections:
- net VBUS: no longer SW1.3 (C)
- no-connect marks 0 -> 1
Changed lines of the file:
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@@
   (junction (at 125.73 104.14) (diameter 0) (color 0 0 0 0)
   )
+  (no_connect (at 132.08 93.98))
   (wire (pts (xy 179.07 91.44) (xy 165.1 91.44))
     (stroke (width 0) (type default))
@@
     (stroke (width 0) (type default))
   )
-  (wire (pts (xy 132.08 93.98) (xy 130.81 93.98))
-    (stroke (width 0) (type default))
-  )
   (wire (pts (xy 114.3 54.61) (xy 147.32 54.61))
     (stroke (width 0) (type default))
@@
   )
   (wire (pts (xy 186.69 60.96) (xy 190.5 60.96))
-    (stroke (width 0) (type default))
-  )
-  (wire (pts (xy 130.81 93.98) (xy 130.81 73.66))
     (stroke (width 0) (type default))
   )
@@
   (text "3.7V LiPo Battery\n" (at 127 114.3 0)
     (effects (font (size 1.27 1.27)) (justify left bottom))
-  )
-  (global_label "VBUS" (shape input) (at 130.81 73.66 90) (fields_autoplaced)
-    (effects (font (size 1.27 1.27)) (justify left))
-    (property "Intersheetrefs" "${INTERSHEET_REFS}" (at 130.81 65.8556 90)
-      (effects (font (size 1.27 1.27)) (justify left) hide)
-    )
   )
   (global_label "VBUS" (shape input) (at 66.04 91.44 180) (fields_autoplaced)
@@
       (effects (font (size 1.27 1.27)) (justify left))
     )
-    (property "Footprint" "Connector_PinHeader_2.54mm:PinHeader_1x02_P2.54mm_Vertical" (at 217.17 82.55 0)
-      (effects (font (size 1.27 1.27)) hide)
-    )
+    (property "Footprint" "Connector_PinSocket_2.54mm:PinSocket_1x02_P2.54mm_Vertical" (at 217.17 82.55 0)
+      (effects (font (size 1.27 1.27)) hide)
+    )
